Commit message: Update: DWA 모듈 완료

File: dwa/urdf/OS1-32.urdf.xacro (robot description, xacro)
@@ -2,5 +2,5 @@
 <robot xmlns:xacro="http://www.ros.org/wiki/xacro" name="OS1-32">
   <xacro:property name="M_PI" value="3.1415926535897931" />
-  <xacro:macro name="OS1-32" params="*origin parent:=base_link name:=os_sensor topic_points:=/ouster/points topic_imu:=/ouster/imu hz:=10 lasers:=32 samples:=1024 min_range:=0.3 max_range:=75.0 noise:=0.008 min_angle:=-${M_PI} max_angle:=${M_PI} lidar_link:=os_lidar imu_link:=os_imu vfov_min:=-.393 vfov_max:=.393">
+  <xacro:macro name="OS1-32" params="*origin parent:=base_link name:=os_sensor topic_points:=/ouster/points topic_imu:=/ouster/imu hz:=10 lasers:=32 samples:=512 min_range:=0.3 max_range:=75.0 noise:=0.008 min_angle:=-${M_PI} max_angle:=${M_PI} lidar_link:=os_lidar imu_link:=os_imu vfov_min:=-.393 vfov_max:=.393 gpu:=true">
     <joint name="${name}_mount_joint" type="fixed">
       <xacro:insert_block name="origin" />
@@ -69,39 +69,76 @@
       <origin xyz="0.0 0.0 0.03618" rpy="0 0 0" />
     </joint>
-    <!-- Gazebo Ouster plugin (built in dwa package) -->
+    <!-- Gazebo Ouster plugin (Gepetto 방식 - GPU 옵션 지원) -->
     <gazebo reference="${name}">
-        <sensor type="gpu_ray" name="${name}-OS1-32">
-          <pose>0 0 0 0 0 0</pose>
-          <visualize>false</visualize>
-          <update_rate>${hz}</update_rate>
-          <ray>
-            <scan>
-              <horizontal>
-                <samples>${samples}</samples>
-                <resolution>1</resolution>
-                <min_angle>${min_angle}</min_angle>
-                <max_angle>${max_angle}</max_angle>
-              </horizontal>
-              <vertical>
-                <samples>${lasers}</samples>
-                <resolution>1</resolution>
-                <min_angle>${vfov_min}</min_angle>
-                <max_angle>${vfov_max}</max_angle>
-              </vertical>
-            </scan>
-            <range>
-              <min>${min_range}</min>
-              <max>${max_range}</max>
-              <resolution>0.03</resolution>
-            </range>
-          </ray>
-          <plugin name="gazebo_ros_laser_controller" filename="libgazebo_ros_ouster_gpu_laser.so">
-            <topicName>${topic_points}</topicName>
-            <frameName>${lidar_link}</frameName>
-            <min_range>${min_range}</min_range>
-            <max_range>${max_range}</max_range>
-            <gaussianNoise>${noise}</gaussianNoise>
-          </plugin>
-        </sensor>
+        <xacro:if value="${gpu}">
+          <sensor type="gpu_ray" name="${name}-OS1-32">
+            <pose>0 0 0 0 0 0</pose>
+            <visualize>false</visualize>
+            <update_rate>${hz}</update_rate>
+            <ray>
+              <scan>
+                <horizontal>
+                  <samples>${samples}</samples>
+                  <resolution>1</resolution>
+                  <min_angle>${min_angle}</min_angle>
+                  <max_angle>${max_angle}</max_angle>
+                </horizontal>
+                <vertical>
+                  <samples>${lasers}</samples>
+                  <resolution>1</resolution>
+                  <min_angle>${vfov_min}</min_angle>
+                  <max_angle>${vfov_max}</max_angle>
+                </vertical>
+              </scan>
+              <range>
+                <min>${min_range}</min>
+                <max>${max_range}</max>
+                <resolution>0.03</resolution>
+              </range>
+            </ray>
+            <plugin name="gazebo_ros_laser_controller" filename="libgazebo_ros_ouster_gpu_laser.so">
+              <topicName>${topic_points}</topicName>
+              <frameName>${lidar_link}</frameName>
+              <min_range>${min_range}</min_range>
+              <max_range>${max_range}</max_range>
+              <gaussianNoise>${noise}</gaussianNoise>
+            </plugin>
+          </sensor>
+        </xacro:if>
+        <xacro:unless value="${gpu}">
+          <sensor type="ray" name="${name}-OS1-32">
+            <pose>0 0 0 0 0 0</pose>
+            <visualize>false</visualize>
+            <update_rate>${hz}</update_rate>
+            <ray>
+              <scan>
+                <horizontal>
+                  <samples>${samples}</samples>
+                  <resolution>1</resolution>
+                  <min_angle>${min_angle}</min_angle>
+                  <max_angle>${max_angle}</max_angle>
+                </horizontal>
+                <vertical>
+                  <samples>${lasers}</samples>
+                  <resolution>1</resolution>
+                  <min_angle>${vfov_min}</min_angle>
+                  <max_angle>${vfov_max}</max_angle>
+                </vertical>
+              </scan>
+              <range>
+                <min>${min_range}</min>
+                <max>${max_range}</max>
+                <resolution>0.03</resolution>
+              </range>
+            </ray>
+            <plugin name="gazebo_ros_laser_controller" filename="libgazebo_ros_ouster_laser.so">
+              <topicName>${topic_points}</topicName>
+              <frameName>${lidar_link}</frameName>
+              <min_range>${min_range}</min_range>
+              <max_range>${max_range}</max_range>
+              <gaussianNoise>${noise}</gaussianNoise>
+            </plugin>
+          </sensor>
+        </xacro:unless>
     </gazebo>
     <!-- IMU -->

File: dwa/urdf/custom_description_ouster_gps.urdf.xacro (robot description, xacro)
@@ -1,28 +1,7 @@
 <?xml version="1.0"?>
-<!--
-Software License Agreement (BSD)
-\file      description.urdf.xacro
-\authors   Paul Bovbel <pbovbel@clearpathrobotics.com>, Devon Ash <dash@clearpathrobotics.com>
-\copyright Copyright (c) 2015, Clearpath Robotics, Inc., All rights reserved.
-Redistribution and use in source and binary forms, with or without modification, are permitted provided that
-the following conditions are met:
- * Redistributions of source code must retain the above copyright notice, this list of conditions and the
-   following disclaimer.
- * Redistributions in binary form must reproduce the above copyright notice, this list of conditions and the
-   following disclaimer in the documentation and/or other materials provided with the distribution.
- * Neither the name of Clearpath Robotics nor the names of its contributors may be used to endorse or promote
-   products derived from this software without specific prior written permission.
-THIS SOFTWARE IS PROVIDED BY THE COPYRIGHT HOLDERS AND CONTRIBUTORS "AS IS" AND ANY EXPRESS OR IMPLIED WAR-
-RANTIES, INCLUDING, BUT NOT LIMITED TO, THE IMPLIED WARRANTIES OF MERCHANTABILITY AND FITNESS FOR A PARTICULAR
-PURPOSE ARE DISCLAIMED. IN NO EVENT SHALL THE COPYRIGHT HOLDER OR CONTRIBUTORS BE LIABLE FOR ANY DIRECT, IN-
-DIRECT, INCIDENTAL, SPECIAL, EXEMPLARY, OR CONSEQUENTIAL DAMAGES (INCLUDING, BUT NOT LIMITED TO, PROCUREMENT
-OF SUBSTITUTE GOODS OR SERVICES; LOSS OF USE, DATA, OR PROFITS; OR BUSINESS INTERRUPTION) HOWEVER CAUSED AND
-ON ANY THEORY OF LIABILITY, WHETHER IN CONTRACT, STRICT LIABILITY, OR TORT (INCLUDING NEGLIGENCE OR OTHERWISE)
-ARISING IN ANY WAY OUT OF THE USE OF THIS SOFTWARE, EVEN IF ADVISED OF THE POSSIBILITY OF SUCH DAMAGE.
--->
 <robot name="husky" xmlns:xacro="http://ros.org/wiki/xacro">
+  <!-- 1) Husky 추가 -->
   <xacro:include filename="$(find husky_description)/urdf/husky.urdf.xacro" />
-  <!-- Insert customization below, sample provided: -->
-  <!-- 2) OS1-64 LiDAR 모델 포함 -->
+  <!-- 2) OS1-64 LiDAR 추가 -->
   <xacro:include filename="$(find dwa)/urdf/OS1-32.urdf.xacro"/>
   <xacro:OS1-32
@@ -43,6 +22,5 @@
     <origin xyz="0.2 0 0.4" rpy="0 0 0"/>
   </xacro:OS1-32>
-   <!-- GPS 추가-->
-  <!-- GPS 센서 포함 -->
+  <!-- 3) GPS 추가 -->
   <!-- <xacro:include filename="$(find dwa)/urdf/gps_sensor.urdf.xacro"/> -->
   <!-- Gazebo 플러그인 포함 -->

File: husky/husky_description/urdf/husky.urdf.xacro (robot description, xacro)
@@ -117,10 +117,12 @@
   <xacro:arg name="outdoornav_configuration" default="$(optenv OUTDOORNAV_CONFIGURATION standard)" />
   <!-- Included URDF/XACRO Files -->
-  <xacro:include filename="$(find husky_description)/urdf/accessories/hokuyo_ust10.urdf.xacro" />
-  <xacro:include filename="$(find husky_description)/urdf/accessories/intel_realsense.urdf.xacro"/>
-  <xacro:include filename="$(find husky_description)/urdf/accessories/flir_blackfly_mount.urdf.xacro"/>
+  <!-- <xacro:include filename="$(find husky_description)/urdf/accessories/hokuyo_ust10.urdf.xacro" />
+  <xacro:include filename="$(find husky_description)/urdf/accessories/intel_realsense.urdf.xacro"/> -->
+  <!-- ❌ Blackfly mount 비활성화: fath_pivot_mount_description, flir_camera_description 패키지 누락 -->
+  <!-- <xacro:include filename="$(find husky_description)/urdf/accessories/flir_blackfly_mount.urdf.xacro"/> -->
   <xacro:include filename="$(find husky_description)/urdf/accessories/sensor_arch.urdf.xacro"/>
-  <xacro:include filename="$(find husky_description)/urdf/accessories/sick_lms1xx_mount.urdf.xacro"/>
-  <xacro:include filename="$(find husky_description)/urdf/accessories/vlp16_mount.urdf.xacro"/>
+  <!-- ❌ SICK LMS1XX mount 비활성화: lms1xx 패키지 누락 -->
+  <!-- <xacro:include filename="$(find husky_description)/urdf/accessories/sick_lms1xx_mount.urdf.xacro"/> -->
+  <!-- <xacro:include filename="$(find husky_description)/urdf/accessories/vlp16_mount.urdf.xacro"/> -->
   <xacro:include filename="$(find husky_description)/urdf/decorations.urdf.xacro" />
   <xacro:include filename="$(find husky_description)/urdf/wheel.urdf.xacro" />
@@ -216,5 +218,6 @@
     SICK LMS1XX Priamry and Secondary Laser Scans
   -->
-  <xacro:if value="$(arg laser_enabled)">
+  <!-- ❌ SICK LMS1XX 비활성화: lms1xx 패키지 누락 -->
+  <!-- <xacro:if value="$(arg laser_enabled)">
     <xacro:sick_lms1xx_mount prefix="$(arg laser_prefix)" parent="$(arg laser_parent)" topic="$(arg laser_topic)" robot_namespace="$(arg robot_namespace)" tower="$(arg laser_tower)">
       <origin xyz="$(arg laser_xyz)" rpy="$(arg laser_rpy)"/>
@@ -225,5 +228,5 @@
       <origin xyz="$(arg laser_secondary_xyz)" rpy="$(arg laser_secondary_rpy)"/>
     </xacro:sick_lms1xx_mount>
-  </xacro:if>
+  </xacro:if> -->
   <!--
     Hokuyo UST10 Primary and Secondary Laser Scans
@@ -275,5 +278,6 @@
   </xacro:if>
   <!-- BlackflyS Camera Primary and Secondary -->
-  <xacro:if value="$(arg blackfly_enabled)">
+  <!-- ❌ Blackfly 사용 비활성화: 패키지 누락으로 주석 처리 -->
+  <!-- <xacro:if value="$(arg blackfly_enabled)">
     <xacro:flir_blackfly_mount prefix="$(arg blackfly_prefix)"
                                 parent="$(arg blackfly_parent)"
@@ -290,5 +294,5 @@
       <origin xyz="$(arg blackfly_secondary_xyz)" rpy="$(arg blackfly_secondary_rpy)"/>
     </xacro:flir_blackfly_mount>
-  </xacro:if>
+  </xacro:if> -->
   <!--
     Velodyne 3D LiDAR Primary and Secondary
@@ -323,8 +327,43 @@
     <xacro:outdoornav_sensors outdoornav_configuration="$(arg outdoornav_configuration)" />
   </xacro:if>
+  <!-- Skid Steer Drive Plugin: 실제 로봇과 동일한 좌/우 차동 구동 방식 -->
+  <!-- 4개 바퀴를 좌/우 2개 그룹으로 제어 (HuskyHardware::writeCommandsToHardware와 동일) -->
   <gazebo>
-    <plugin name="gazebo_ros_control" filename="libgazebo_ros_control.so">
+    <plugin name="skid_steer_drive_controller" filename="libgazebo_ros_skid_steer_drive.so">
+      <updateRate>100.0</updateRate>
       <robotNamespace>$(arg robot_namespace)</robotNamespace>
-      <legacyModeNS>true</legacyModeNS>
+      <!-- 좌측 바퀴 2개 -->
+      <leftFrontJoint>front_left_wheel</leftFrontJoint>
+      <leftRearJoint>rear_left_wheel</leftRearJoint>
+      <!-- 우측 바퀴 2개 -->
+      <rightFrontJoint>front_right_wheel</rightFrontJoint>
+      <rightRearJoint>rear_right_wheel</rightRearJoint>
+      <!-- 바퀴 간격 및 직경 (control.yaml과 일치) -->
+      <wheelSeparation>0.5708</wheelSeparation>
+      <wheelDiameter>0.3302</wheelDiameter>
+      <!-- 토크 및 속도 제한 -->
+      <torque>200</torque>
+      <commandTopic>husky_velocity_controller/cmd_vel</commandTopic>
+      <odometryTopic>husky_velocity_controller/odom</odometryTopic>
+      <odometryFrame>odom</odometryFrame>
+      <robotBaseFrame>base_link</robotBaseFrame>
+      <!-- 공분산 설정 (control.yaml과 일치) -->
+      <covariance_x>0.001</covariance_x>
+      <covariance_y>0.001</covariance_y>
+      <covariance_yaw>0.03</covariance_yaw>
+      <broadcastTF>true</broadcastTF>
+      <publishWheelTF>false</publishWheelTF>
+      <publishWheelJointState>false</publishWheelJointState>
+      <legacyMode>false</legacyMode>
+      <alwaysOn>true</alwaysOn>
+    </plugin>
+  </gazebo>
+  <!-- Joint State Publisher Plugin: 바퀴 4개의 joint_state 발행 (TF 생성용) -->
+  <!-- 실제 로봇의 엔코더 피드백과 동일한 역할 -->
+  <gazebo>
+    <plugin name="joint_state_publisher" filename="libgazebo_ros_joint_state_publisher.so">
+      <robotNamespace>$(arg robot_namespace)</robotNamespace>
+      <jointName>front_left_wheel, front_right_wheel, rear_left_wheel, rear_right_wheel</jointName>
+      <updateRate>50.0</updateRate>
     </plugin>
   </gazebo>

File: husky/husky_description/urdf/wheel.urdf.xacro (robot description, xacro)
@@ -55,5 +55,7 @@
 			<axis xyz="0 1 0" rpy="0 0 0" />
 		</joint>
-		<transmission name="${wheel_prefix}_wheel_trans" type="SimpleTransmission">
+		<!-- Transmission 제거: Gazebo Skid Steer Plugin이 직접 바퀴 제어 -->
+		<!-- 실제 로봇과 동일하게 좌/우 2개 속도로 4개 바퀴 제어 -->
+		<!-- <transmission name="${wheel_prefix}_wheel_trans" type="SimpleTransmission">
 			<type>transmission_interface/SimpleTransmission</type>
 			<actuator name="${wheel_prefix}_wheel_motor">
@@ -63,5 +65,5 @@
 				<hardwareInterface>hardware_interface/VelocityJointInterface</hardwareInterface>
 			</joint>
-		</transmission>
+		</transmission> -->
 	</xacro:macro>
 </robot>
