Commit message: Update: DWA 모듈 완료

File: dwa/urdf/custom_description.gazebo.xacro (robot description, xacro)
@@ -26,10 +26,28 @@
   <xacro:arg name="kinect_enabled" default="false" />
   <!-- Gazebo plugin for ROS Control -->
-  <!-- <gazebo>
+  <gazebo>
     <plugin name="gazebo_ros_control" filename="libgazebo_ros_control.so">
       <robotNamespace>/</robotNamespace>
+      <robotSimType>gazebo_ros_control/DefaultRobotHWSim</robotSimType>
+      <legacyModeNS>true</legacyModeNS>
     </plugin>
-  </gazebo> -->
-  <!-- <xacro:husky_robot_gazebo /> -->
+  </gazebo>
+  <!-- Transmissions for ros_control -->
+  <xacro:macro name="wheel_transmission" params="name">
+    <transmission name="${name}_transmission">
+      <type>transmission_interface/SimpleTransmission</type>
+      <joint name="${name}">
+        <hardwareInterface>hardware_interface/VelocityJointInterface</hardwareInterface>
+      </joint>
+      <actuator name="${name}_actuator">
+        <mechanicalReduction>1</mechanicalReduction>
+      </actuator>
+    </transmission>
+  </xacro:macro>
+  <!-- Apply transmissions to all wheels -->
+  <xacro:wheel_transmission name="front_left_wheel"/>
+  <xacro:wheel_transmission name="front_right_wheel"/>
+  <xacro:wheel_transmission name="rear_left_wheel"/>
+  <xacro:wheel_transmission name="rear_right_wheel"/>
   <gazebo>
     <plugin name="gps_sim" filename="libhector_gazebo_ros_gps.so">

File: dwa/urdf/custom_description_ouster_gps.urdf.xacro (robot description, xacro)
@@ -24,5 +24,5 @@
   <!-- 3) GPS 추가 -->
   <!-- <xacro:include filename="$(find dwa)/urdf/gps_sensor.urdf.xacro"/> -->
-  <!-- Gazebo 플러그인 포함 -->
-  <!-- <xacro:include filename="$(find dwa)/urdf/custom_description.gazebo.xacro"/> -->
+  <!-- Gazebo 플러그인 포함 (ros_control + GPS) -->
+  <xacro:include filename="$(find dwa)/urdf/custom_description.gazebo.xacro"/>
 </robot>
