Commit message: Update: robot_description

File: robot_description/urdf/OS1-32.urdf.xacro (robot description, xacro)
@@ -50,5 +50,5 @@
          <origin xyz="0 0 0.0" rpy="0 0 1.5707"/>
          <geometry>
-	         <mesh filename="package://ouster_description/meshes/os1_64.dae"/>
+	         <mesh filename="package://robot_description/meshes/os1_64.dae"/>
            <!-- <cylinder length="0.073" radius="0.04"/> -->
          </geometry>

File: robot_description/urdf/custom_description.urdf.xacro (robot description, xacro)
@@ -5,4 +5,7 @@
   <!-- 2) OS1-32 LiDAR 추가 -->
   <xacro:include filename="$(find robot_description)/urdf/OS1-32.urdf.xacro"/>
+  <xacro:OS1-32 parent="top_plate_link">
+    <origin xyz="0.0 0.0 0.0" rpy="0 0 0"/>
+  </xacro:OS1-32>
   <!-- 3) GPS 추가 -->
   <xacro:include filename="$(find robot_description)/urdf/gps.urdf.xacro"/>

File: robot_description/urdf/gps.urdf.xacro (robot description, xacro)
@@ -14,5 +14,7 @@
         <box size="0.05 0.05 0.02"/>
       </geometry>
-      <material name="black"/>
+      <material name="black">
+        <color rgba="0.1 0.1 0.1 1.0"/>
+      </material>
     </visual>
     <collision>
