Commit message: dwa 수정 중: 경로만 개선할 것 (동작은 O)

File: robot_description/urdf/custom_description.urdf.xacro (robot description, xacro)
@@ -11,17 +11,17 @@
   <!-- 3) GPS 추가 -->
   <xacro:include filename="$(find robot_description)/urdf/gps.urdf.xacro"/>
-  <!-- 4) Husky Differential Drive Plugin (Custom) -->
+  <!-- 4) Husky Differential Drive Plugin (Gazebo 표준) -->
   <gazebo>
-    <plugin name="husky_diff_drive" filename="libhusky_gazebo_plugin.so">
+    <plugin name="differential_drive_controller" filename="libgazebo_ros_diff_drive.so">
+      <updateRate>50.0</updateRate>
       <!-- Wheel joints -->
-      <leftFrontJoint>front_left_wheel</leftFrontJoint>
-      <leftRearJoint>rear_left_wheel</leftRearJoint>
-      <rightFrontJoint>front_right_wheel</rightFrontJoint>
-      <rightRearJoint>rear_right_wheel</rightRearJoint>
-      <!-- Robot physical parameters (실제 허스키와 동일) -->
+      <leftJoint>front_left_wheel</leftJoint>
+      <leftJoint>rear_left_wheel</leftJoint>
+      <rightJoint>front_right_wheel</rightJoint>
+      <rightJoint>rear_right_wheel</rightJoint>
+      <!-- Kinematics -->
       <wheelSeparation>0.5708</wheelSeparation>
       <wheelDiameter>0.3302</wheelDiameter>
-      <!-- Update rate -->
-      <updateRate>50.0</updateRate>
+      <wheelTorque>200</wheelTorque>
       <!-- Topics -->
       <commandTopic>husky_velocity_controller/cmd_vel</commandTopic>
@@ -30,6 +30,8 @@
       <odometryFrame>odom</odometryFrame>
       <robotBaseFrame>base_link</robotBaseFrame>
-      <!-- Publish odom TF: Gazebo ground truth -->
+      <!-- Publish odom TF -->
       <publishOdomTF>true</publishOdomTF>
+      <publishWheelTF>false</publishWheelTF>
+      <publishWheelJointState>false</publishWheelJointState>
     </plugin>
   </gazebo>

File: robot_description/urdf/gps.urdf.xacro (robot description, xacro)
@@ -27,5 +27,5 @@
   <!-- GPS Joint: top_plate_link에서 60cm 위로 -->
   <joint name="gps_joint" type="fixed">
-    <origin xyz="0.0 0.0 0.6" rpy="0 0 0"/>
+    <origin xyz="0.0 0.0 0.4" rpy="0 0 0"/>
     <parent link="top_plate_link"/>
     <child link="gps_link"/>
