Commit message: 리팩토링 재시작

File: husky/husky_description/urdf/wheel.urdf.xacro (robot description, xacro)
@@ -55,7 +55,5 @@
 			<axis xyz="0 1 0" rpy="0 0 0" />
 		</joint>
-		<!-- Transmission 제거: Gazebo Skid Steer Plugin이 직접 바퀴 제어 -->
-		<!-- 실제 로봇과 동일하게 좌/우 2개 속도로 4개 바퀴 제어 -->
-		<!-- <transmission name="${wheel_prefix}_wheel_trans" type="SimpleTransmission">
+		<transmission name="${wheel_prefix}_wheel_trans" type="SimpleTransmission">
 			<type>transmission_interface/SimpleTransmission</type>
 			<actuator name="${wheel_prefix}_wheel_motor">
@@ -65,5 +63,5 @@
 				<hardwareInterface>hardware_interface/VelocityJointInterface</hardwareInterface>
 			</joint>
-		</transmission> -->
+		</transmission>
 	</xacro:macro>
 </robot>

Commit message: 허스키 urdf 최소화

File: husky/husky_description/urdf/husky.urdf.xacro (robot description, xacro)
@@ -102,6 +102,6 @@
   <xacro:arg name="blackfly_secondary_rpy"            default="$(optenv HUSKY_BLACKFLY_SECONDARY_RPY 0 0 0)"/> -->
   <!-- Bumper Extension -->
-  <!-- <xacro:property name="husky_front_bumper_extend"  value="$(optenv HUSKY_FRONT_BUMPER_EXTEND 0)" />
-  <xacro:property name="husky_rear_bumper_extend"   value="$(optenv HUSKY_REAR_BUMPER_EXTEND 0)" /> -->
+  <xacro:property name="husky_front_bumper_extend"  value="$(optenv HUSKY_FRONT_BUMPER_EXTEND 0)" />
+  <xacro:property name="husky_rear_bumper_extend"   value="$(optenv HUSKY_REAR_BUMPER_EXTEND 0)" />
   <!-- Height of the sensor arch in mm.  Must be either 510 or 300 -->
   <!-- <xacro:arg name="sensor_arch"         default="$(optenv HUSKY_SENSOR_ARCH 0)" />
@@ -110,10 +110,10 @@
   <xacro:arg name="sensor_arch_rpy"     default="$(optenv HUSKY_SENSOR_ARCH_RPY 0 0 0)"/> -->
   <!-- Extras -->
-  <!-- <xacro:arg name="robot_namespace" default="$(optenv ROBOT_NAMESPACE /)" />
+  <xacro:arg name="robot_namespace" default="$(optenv ROBOT_NAMESPACE /)" />
   <xacro:arg name="urdf_extras"     default="$(optenv HUSKY_URDF_EXTRAS empty.urdf)" />
-  <xacro:arg name="cpr_urdf_extras" default="$(optenv CPR_URDF_EXTRAS empty.urdf)" /> -->
+  <xacro:arg name="cpr_urdf_extras" default="$(optenv CPR_URDF_EXTRAS empty.urdf)" />
   <!-- OutdoorNav -->
-  <!-- <xacro:arg name="outdoornav_enabled"       default="$(optenv OUTDOORNAV_ENABLED 0)" />
-  <xacro:arg name="outdoornav_configuration" default="$(optenv OUTDOORNAV_CONFIGURATION standard)" /> -->
+  <xacro:arg name="outdoornav_enabled"       default="$(optenv OUTDOORNAV_ENABLED 0)" />
+  <xacro:arg name="outdoornav_configuration" default="$(optenv OUTDOORNAV_CONFIGURATION standard)" />
   <!-- Included URDF/XACRO Files -->
   <!-- <xacro:include filename="$(find husky_description)/urdf/accessories/hokuyo_ust10.urdf.xacro" />
@@ -122,6 +122,6 @@
   <xacro:include filename="$(find husky_description)/urdf/accessories/sensor_arch.urdf.xacro"/>
   <xacro:include filename="$(find husky_description)/urdf/accessories/sick_lms1xx_mount.urdf.xacro"/>
-  <xacro:include filename="$(find husky_description)/urdf/accessories/vlp16_mount.urdf.xacro"/>
-  <xacro:include filename="$(find husky_description)/urdf/decorations.urdf.xacro" /> -->
+  <xacro:include filename="$(find husky_description)/urdf/accessories/vlp16_mount.urdf.xacro"/> -->
+  <xacro:include filename="$(find husky_description)/urdf/decorations.urdf.xacro" />
   <xacro:include filename="$(find husky_description)/urdf/wheel.urdf.xacro" />
   <xacro:property name="M_PI" value="3.14159"/>
@@ -159,12 +159,12 @@
   </link>
   <!-- Base footprint is on the ground under the robot -->
-  <link name="base_footprint"/>
+  <!-- <link name="base_footprint"/>
   <joint name="base_footprint_joint" type="fixed">
     <origin xyz="0 0 ${wheel_vertical_offset - wheel_radius}" rpy="0 0 0" />
     <parent link="base_link" />
     <child link="base_footprint" />
-  </joint>
+  </joint> -->
   <!-- Inertial link stores the robot's inertial information -->
-  <link name="inertial_link">
+  <!-- <link name="inertial_link">
     <inertial>
       <mass value="46.034" />
@@ -177,5 +177,5 @@
     <parent link="base_link" />
     <child link="inertial_link" />
-  </joint>
+  </joint> -->
   <!-- Husky wheel macros -->
   <xacro:husky_wheel wheel_prefix="front_left">
@@ -192,5 +192,5 @@
   </xacro:husky_wheel>
   <!-- Husky Decorations -->
-  <!-- <xacro:husky_decorate /> -->
+  <xacro:husky_decorate />
   <!--
     Add the main sensor arch if the user has specifically enabled it, or if a sensor
@@ -322,6 +322,6 @@
     <xacro:include filename="$(find cpr_onav_description)/urdf/outdoornav_description.urdf.xacro" />
     <xacro:outdoornav_sensors outdoornav_configuration="$(arg outdoornav_configuration)" />
-  </xacro:if>
-  <gazebo>
+  </xacro:if> -->
+  <!-- <gazebo>
     <plugin name="gazebo_ros_control" filename="libgazebo_ros_control.so">
       <robotNamespace>$(arg robot_namespace)</robotNamespace>

Commit message: Update: 가제보 로드 성공

File: husky/husky_description/urdf/husky.urdf.xacro (robot description, xacro)
@@ -166,5 +166,5 @@
   </joint> -->
   <!-- Inertial link stores the robot's inertial information -->
-  <!-- <link name="inertial_link">
+  <link name="inertial_link">
     <inertial>
       <mass value="46.034" />
@@ -177,5 +177,5 @@
     <parent link="base_link" />
     <child link="inertial_link" />
-  </joint> -->
+  </joint>
   <!-- Husky wheel macros -->
   <xacro:husky_wheel wheel_prefix="front_left">

File: robot_description/urdf/custom_description.urdf.xacro (robot description, xacro)
@@ -6,7 +6,40 @@
   <xacro:include filename="$(find robot_description)/urdf/OS1-32.urdf.xacro"/>
   <xacro:OS1-32 parent="top_plate_link">
-    <origin xyz="0.0 0.0 0.0" rpy="0 0 0"/>
+    <!-- front_wheel 쪽으로 이동 + 60cm 위로 -->
+    <origin xyz="0.3 0.0 0.6" rpy="0 0 0"/>
   </xacro:OS1-32>
   <!-- 3) GPS 추가 -->
   <xacro:include filename="$(find robot_description)/urdf/gps.urdf.xacro"/>
+  <!-- 4) Husky Differential Drive Plugin -->
+  <gazebo>
+    <plugin name="husky_diff_drive" filename="libhusky_gazebo_plugin.so">
+      <!-- Wheel joints -->
+      <leftFrontJoint>front_left_wheel</leftFrontJoint>
+      <leftRearJoint>rear_left_wheel</leftRearJoint>
+      <rightFrontJoint>front_right_wheel</rightFrontJoint>
+      <rightRearJoint>rear_right_wheel</rightRearJoint>
+      <!-- Robot physical parameters (실제 허스키와 동일) -->
+      <wheelSeparation>0.5708</wheelSeparation>
+      <wheelDiameter>0.3302</wheelDiameter>
+      <!-- Update rate -->
+      <updateRate>50.0</updateRate>
+      <!-- Topics -->
+      <commandTopic>husky_velocity_controller/cmd_vel</commandTopic>
+      <odometryTopic>husky_velocity_controller/odom</odometryTopic>
+      <!-- Frames -->
+      <odometryFrame>odom</odometryFrame>
+      <robotBaseFrame>base_link</robotBaseFrame>
+      <!-- Publish odom TF: false (robot_localization이 발행) -->
+      <publishOdomTF>false</publishOdomTF>
+    </plugin>
+  </gazebo>
+  <!-- 5) Joint State Publisher Plugin -->
+  <gazebo>
+    <plugin name="joint_state_publisher" filename="libgazebo_ros_joint_state_publisher.so">
+      <robotNamespace>/</robotNamespace>
+      <jointName>front_left_wheel, front_right_wheel, rear_left_wheel, rear_right_wheel</jointName>
+      <updateRate>50.0</updateRate>
+      <alwaysOn>true</alwaysOn>
+    </plugin>
+  </gazebo>
 </robot>

File: robot_description/urdf/gps.urdf.xacro (robot description, xacro)
@@ -4,16 +4,16 @@
   <link name="gps_link">
     <inertial>
-      <mass value="0.001"/>
+      <mass value="0.01"/>
       <origin xyz="0 0 0" rpy="0 0 0"/>
-      <inertia ixx="0.000000017" ixy="0" ixz="0"
-               iyy="0.000000017" iyz="0" izz="0.000000017"/>
+      <inertia ixx="0.00001" ixy="0" ixz="0"
+               iyy="0.00001" iyz="0" izz="0.00001"/>
     </inertial>
     <visual>
       <origin xyz="0 0 0" rpy="0 0 0"/>
       <geometry>
-        <box size="0.05 0.05 0.02"/>
+        <box size="0.15 0.15 0.05"/>
       </geometry>
-      <material name="black">
-        <color rgba="0.1 0.1 0.1 1.0"/>
+      <material name="gps_red">
+        <color rgba="1.0 0.0 0.0 1.0"/>
       </material>
     </visual>
@@ -21,13 +21,35 @@
       <origin xyz="0 0 0" rpy="0 0 0"/>
       <geometry>
-        <box size="0.05 0.05 0.02"/>
+        <box size="0.15 0.15 0.05"/>
       </geometry>
     </collision>
   </link>
-  <!-- GPS Joint -->
+  <!-- GPS Joint: top_plate_link에서 60cm 위로 -->
   <joint name="gps_joint" type="fixed">
-    <origin xyz="0.0 0.0 0.1" rpy="0 0 0"/>
-    <parent link="base_link"/>
+    <origin xyz="0.0 0.0 0.6" rpy="0 0 0"/>
+    <parent link="top_plate_link"/>
     <child link="gps_link"/>
   </joint>
+  <!-- Gazebo GPS material -->
+  <gazebo reference="gps_link">
+    <material>Gazebo/Red</material>
+  </gazebo>
+  <!-- Gazebo GPS Plugin -->
+  <gazebo>
+    <plugin name="gazebo_ros_gps" filename="libhector_gazebo_ros_gps.so">
+      <updateRate>10.0</updateRate>
+      <bodyName>gps_link</bodyName>
+      <frameId>gps_link</frameId>
+      <topicName>/ublox/fix</topicName>
+      <velocityTopicName>/ublox/fix_velocity</velocityTopicName>
+      <referenceLatitude>0.0</referenceLatitude>
+      <referenceLongitude>0.0</referenceLongitude>
+      <referenceHeading>0.0</referenceHeading>
+      <referenceAltitude>0.0</referenceAltitude>
+      <drift>0.001 0.001 0.001</drift>
+      <gaussianNoise>0.01 0.01 0.01</gaussianNoise>
+      <velocityDrift>0.001 0.001 0.001</velocityDrift>
+      <velocityGaussianNoise>0.05 0.05 0.05</velocityGaussianNoise>
+    </plugin>
+  </gazebo>
 </robot>
