Commit message: faster-lio 시뮬레이션 버그 해결

File: oss/husky/husky_description/urdf/husky.urdf.xacro (robot description, xacro)
@@ -23,9 +23,9 @@
 <robot name="husky" xmlns:xacro="http://ros.org/wiki/xacro">
   <!-- IMU Link -->
-  <!-- <xacro:arg name="imu_xyz"     default="$(optenv HUSKY_IMU_XYZ 0.19 0 0.149)"/>
+  <xacro:arg name="imu_xyz"     default="$(optenv HUSKY_IMU_XYZ 0.19 0 0.149)"/>
   <xacro:arg name="imu_rpy"     default="$(optenv HUSKY_IMU_RPY 0 -1.5708 3.1416)"/>
-  <xacro:arg name="imu_parent"  default="$(optenv HUSKY_IMU_PARENT base_link)"/> -->
+  <xacro:arg name="imu_parent"  default="$(optenv HUSKY_IMU_PARENT base_link)"/>
   <!-- LMS1XX Laser Primary and Secondary -->
-  <!-- <xacro:arg name="laser_enabled"           default="$(optenv HUSKY_LMS1XX_ENABLED 0)" />
+  <xacro:arg name="laser_enabled"           default="$(optenv HUSKY_LMS1XX_ENABLED 0)" />
   <xacro:arg name="laser_topic"             default="$(optenv HUSKY_LMS1XX_TOPIC front/scan)"/>
   <xacro:arg name="laser_tower"             default="$(optenv HUSKY_LMS1XX_TOWER 1)"/>
@@ -40,7 +40,7 @@
   <xacro:arg name="laser_secondary_parent"  default="$(optenv HUSKY_LMS1XX_SECONDARY_PARENT top_plate_link)"/>
   <xacro:arg name="laser_secondary_xyz"     default="$(optenv HUSKY_LMS1XX_SECONDARY_XYZ -0.2206 0.0 0.00635)" />
-  <xacro:arg name="laser_secondary_rpy"     default="$(optenv HUSKY_LMS1XX_SECONDARY_RPY 0.0 0.0 3.14159)" /> -->
+  <xacro:arg name="laser_secondary_rpy"     default="$(optenv HUSKY_LMS1XX_SECONDARY_RPY 0.0 0.0 3.14159)" />
   <!-- UST10 Laser Primary  and Secondary -->
-  <!-- <xacro:arg name="laser_ust10_front_enabled" default="$(optenv HUSKY_UST10_ENABLED 0)" />
+  <xacro:arg name="laser_ust10_front_enabled" default="$(optenv HUSKY_UST10_ENABLED 0)" />
   <xacro:arg name="laser_ust10_front_topic"   default="$(optenv HUSKY_UST10_TOPIC front/scan)" />
   <xacro:arg name="laser_ust10_front_prefix"  default="$(optenv HUSKY_UST10_PREFIX front)" />
@@ -53,7 +53,7 @@
   <xacro:arg name="laser_ust10_rear_parent"   default="$(optenv HUSKY_UST10_SECONDARY_PARENT top_plate_link)" />
   <xacro:arg name="laser_ust10_rear_xyz"      default="$(optenv HUSKY_UST10_SECONDARY_XYZ -0.2206 0.0 0.00635)" />
-  <xacro:arg name="laser_ust10_rear_rpy"      default="$(optenv HUSKY_UST10_SECONDARY_RPY 0 0 3.14159)" /> -->
+  <xacro:arg name="laser_ust10_rear_rpy"      default="$(optenv HUSKY_UST10_SECONDARY_RPY 0 0 3.14159)" />
   <!-- Velodyne LiDAR Primary and Secondary -->
-  <!-- <xacro:arg name="laser_3d_enabled"              default="$(optenv HUSKY_LASER_3D_ENABLED 0)" />
+  <xacro:arg name="laser_3d_enabled"              default="$(optenv HUSKY_LASER_3D_ENABLED 0)" />
   <xacro:arg name="laser_3d_topic"                default="$(optenv HUSKY_LASER_3D_TOPIC points)"/>
   <xacro:arg name="laser_3d_tower"                default="$(optenv HUSKY_LASER_3D_TOWER 1)"/>
@@ -68,7 +68,7 @@
   <xacro:arg name="laser_3d_secondary_parent"     default="$(optenv HUSKY_LASER_3D_SECONDARY_PARENT top_plate_link)"/>
   <xacro:arg name="laser_3d_secondary_xyz"        default="$(optenv HUSKY_LASER_3D_SECONDARY_XYZ 0 0 0)" />
-  <xacro:arg name="laser_3d_secondary_rpy"        default="$(optenv HUSKY_LASER_3D_SECONDARY_RPY 0 0 -3.14159)" /> -->
+  <xacro:arg name="laser_3d_secondary_rpy"        default="$(optenv HUSKY_LASER_3D_SECONDARY_RPY 0 0 -3.14159)" />
   <!-- Realsense Camera Primary and Secondary -->
-  <!-- <xacro:arg name="realsense_enabled"             default="$(optenv HUSKY_REALSENSE_ENABLED 0)" />
+  <xacro:arg name="realsense_enabled"             default="$(optenv HUSKY_REALSENSE_ENABLED 0)" />
   <xacro:arg name="realsense_model"               default="$(optenv HUSKY_REALSENSE_MODEL d435)"/>
   <xacro:arg name="realsense_topic"               default="$(optenv HUSKY_REALSENSE_TOPIC realsense)" />
@@ -85,7 +85,7 @@
   <xacro:arg name="realsense_secondary_xyz"       default="$(optenv HUSKY_REALSENSE_SECONDARY_XYZ 0 0 0)" />
   <xacro:arg name="realsense_secondary_rpy"       default="$(optenv HUSKY_REALSENSE_SECONDARY_RPY 0 0 0)" />
-  <xacro:property name="realsense_secondary_model" value="$(arg realsense_secondary_model)"/> -->
+  <xacro:property name="realsense_secondary_model" value="$(arg realsense_secondary_model)"/>
   <!-- BlackflyS Camera Primary and Secondary -->
-  <!-- <xacro:arg name="blackfly_enabled"                  default="$(optenv HUSKY_BLACKFLY 0)"/>
+  <xacro:arg name="blackfly_enabled"                  default="$(optenv HUSKY_BLACKFLY 0)"/>
   <xacro:arg name="blackfly_mount_enabled"            default="$(optenv HUSKY_BLACKFLY_MOUNT_ENABLED 1)"/>
   <xacro:arg name="blackfly_mount_angle"              default="$(optenv HUSKY_BLACKFLY_MOUNT_ANGLE 0)"/>
@@ -100,13 +100,13 @@
   <xacro:arg name="blackfly_secondary_parent"         default="$(optenv HUSKY_BLACKFLY_SECONDARY_PARENT top_plate_link)"/>
   <xacro:arg name="blackfly_secondary_xyz"            default="$(optenv HUSKY_BLACKFLY_SECONDARY_XYZ 0 0 0)"/>
-  <xacro:arg name="blackfly_secondary_rpy"            default="$(optenv HUSKY_BLACKFLY_SECONDARY_RPY 0 0 0)"/> -->
+  <xacro:arg name="blackfly_secondary_rpy"            default="$(optenv HUSKY_BLACKFLY_SECONDARY_RPY 0 0 0)"/>
   <!-- Bumper Extension -->
   <xacro:property name="husky_front_bumper_extend"  value="$(optenv HUSKY_FRONT_BUMPER_EXTEND 0)" />
   <xacro:property name="husky_rear_bumper_extend"   value="$(optenv HUSKY_REAR_BUMPER_EXTEND 0)" />
   <!-- Height of the sensor arch in mm.  Must be either 510 or 300 -->
-  <!-- <xacro:arg name="sensor_arch"         default="$(optenv HUSKY_SENSOR_ARCH 0)" />
+  <xacro:arg name="sensor_arch"         default="$(optenv HUSKY_SENSOR_ARCH 0)" />
   <xacro:arg name="sensor_arch_height"  default="$(optenv HUSKY_SENSOR_ARCH_HEIGHT 510)" />
   <xacro:arg name="sensor_arch_xyz"     default="$(optenv HUSKY_SENSOR_ARCH_OFFSET 0 0 0)"/>
-  <xacro:arg name="sensor_arch_rpy"     default="$(optenv HUSKY_SENSOR_ARCH_RPY 0 0 0)"/> -->
+  <xacro:arg name="sensor_arch_rpy"     default="$(optenv HUSKY_SENSOR_ARCH_RPY 0 0 0)"/>
   <!-- Extras -->
   <xacro:arg name="robot_namespace" default="$(optenv ROBOT_NAMESPACE /)" />
@@ -118,9 +118,11 @@
   <!-- Included URDF/XACRO Files -->
   <!-- <xacro:include filename="$(find husky_description)/urdf/accessories/hokuyo_ust10.urdf.xacro" />
-  <xacro:include filename="$(find husky_description)/urdf/accessories/intel_realsense.urdf.xacro"/>
-  <xacro:include filename="$(find husky_description)/urdf/accessories/flir_blackfly_mount.urdf.xacro"/>
+  <xacro:include filename="$(find husky_description)/urdf/accessories/intel_realsense.urdf.xacro"/> -->
+  <!-- ❌ Blackfly mount 비활성화: fath_pivot_mount_description, flir_camera_description 패키지 누락 -->
+  <!-- <xacro:include filename="$(find husky_description)/urdf/accessories/flir_blackfly_mount.urdf.xacro"/> -->
   <xacro:include filename="$(find husky_description)/urdf/accessories/sensor_arch.urdf.xacro"/>
-  <xacro:include filename="$(find husky_description)/urdf/accessories/sick_lms1xx_mount.urdf.xacro"/>
-  <xacro:include filename="$(find husky_description)/urdf/accessories/vlp16_mount.urdf.xacro"/> -->
+  <!-- ❌ SICK LMS1XX mount 비활성화: lms1xx 패키지 누락 -->
+  <!-- <xacro:include filename="$(find husky_description)/urdf/accessories/sick_lms1xx_mount.urdf.xacro"/> -->
+  <!-- <xacro:include filename="$(find husky_description)/urdf/accessories/vlp16_mount.urdf.xacro"/> -->
   <xacro:include filename="$(find husky_description)/urdf/decorations.urdf.xacro" />
   <xacro:include filename="$(find husky_description)/urdf/wheel.urdf.xacro" />
@@ -132,5 +134,5 @@
   <!-- Wheel Mounting Positions -->
   <xacro:property name="wheelbase" value="0.5120" />
-  <xacro:property name="track" value="0.555" />
+  <xacro:property name="track" value="0.5708" />
   <xacro:property name="wheel_vertical_offset" value="0.03282" />
   <!-- Wheel Properties -->
@@ -159,10 +161,10 @@
   </link>
   <!-- Base footprint is on the ground under the robot -->
-  <!-- <link name="base_footprint"/>
+  <link name="base_footprint"/>
   <joint name="base_footprint_joint" type="fixed">
     <origin xyz="0 0 ${wheel_vertical_offset - wheel_radius}" rpy="0 0 0" />
     <parent link="base_link" />
     <child link="base_footprint" />
-  </joint> -->
+  </joint>
   <!-- Inertial link stores the robot's inertial information -->
   <link name="inertial_link">
@@ -197,13 +199,13 @@
     requires it for mounting
   -->
-  <!-- <xacro:if value="$(arg sensor_arch)">
+  <xacro:if value="$(arg sensor_arch)">
     <xacro:sensor_arch prefix="" parent="top_plate_link" size="$(arg sensor_arch_height)">
       <origin xyz="$(arg sensor_arch_xyz)" rpy="$(arg sensor_arch_rpy)"/>
     </xacro:sensor_arch>
-  </xacro:if> -->
+  </xacro:if>
   <!--
       IMU Link: Standard location to add an IMU (i.e. UM7 or Microstrain)
   -->
-  <!-- <link name="imu_link"/>
+  <link name="imu_link"/>
   <joint name="imu_joint" type="fixed">
     <origin xyz="$(arg imu_xyz)" rpy="$(arg imu_rpy)" />
@@ -212,8 +214,9 @@
   </joint>
   <gazebo reference="imu_link">
-  </gazebo> -->
+  </gazebo>
   <!--
     SICK LMS1XX Priamry and Secondary Laser Scans
   -->
+  <!-- ❌ SICK LMS1XX 비활성화: lms1xx 패키지 누락 -->
   <!-- <xacro:if value="$(arg laser_enabled)">
     <xacro:sick_lms1xx_mount prefix="$(arg laser_prefix)" parent="$(arg laser_parent)" topic="$(arg laser_topic)" robot_namespace="$(arg robot_namespace)" tower="$(arg laser_tower)">
@@ -229,5 +232,5 @@
     Hokuyo UST10 Primary and Secondary Laser Scans
   -->
-  <!-- <xacro:if value="$(arg laser_ust10_front_enabled)">
+  <xacro:if value="$(arg laser_ust10_front_enabled)">
     <xacro:hokuyo_ust10_mount topic="$(arg laser_ust10_front_topic)" prefix="$(arg laser_ust10_front_prefix)" parent_link="$(arg laser_ust10_front_parent)">
         <origin xyz="$(arg laser_ust10_front_xyz)" rpy="$(arg laser_ust10_front_rpy)" />
@@ -238,7 +241,7 @@
         <origin xyz="$(arg laser_ust10_rear_xyz)" rpy="$(arg laser_ust10_rear_rpy)" />
       </xacro:hokuyo_ust10_mount>
-  </xacro:if> -->
+  </xacro:if>
   <!-- Intel Realsense Primary and Secondary -->
-  <!-- <xacro:property name="realsense_enabled" value="$(arg realsense_enabled)"/>
+  <xacro:property name="realsense_enabled" value="$(arg realsense_enabled)"/>
   <xacro:property name="realsense_secondary_enabled" value="$(arg realsense_secondary_enabled)"/>
   <xacro:if value="${realsense_enabled or realsense_secondary_enabled}">
@@ -273,6 +276,7 @@
       <origin xyz="$(arg realsense_secondary_xyz)" rpy="$(arg realsense_secondary_rpy)"/>
     </xacro:realsense_sensor>
-  </xacro:if> -->
+  </xacro:if>
   <!-- BlackflyS Camera Primary and Secondary -->
+  <!-- ❌ Blackfly 사용 비활성화: 패키지 누락으로 주석 처리 -->
   <!-- <xacro:if value="$(arg blackfly_enabled)">
     <xacro:flir_blackfly_mount prefix="$(arg blackfly_prefix)"
@@ -294,5 +298,5 @@
     Velodyne 3D LiDAR Primary and Secondary
   -->
-  <!-- <xacro:if value="$(arg laser_3d_enabled)">
+  <xacro:if value="$(arg laser_3d_enabled)">
     <xacro:if value="$(arg laser_3d_tower)">
       <xacro:vlp16_mount prefix="$(arg laser_3d_prefix)" parent_link="$(arg laser_3d_parent)" topic="$(arg laser_3d_topic)">
@@ -317,11 +321,11 @@
       </xacro:VLP-16>
     </xacro:unless>
-  </xacro:if> -->
+  </xacro:if>
   <!-- OutdoorNav URDF Config -->
-  <!-- <xacro:if value="$(arg outdoornav_enabled)">
+  <xacro:if value="$(arg outdoornav_enabled)">
     <xacro:include filename="$(find cpr_onav_description)/urdf/outdoornav_description.urdf.xacro" />
     <xacro:outdoornav_sensors outdoornav_configuration="$(arg outdoornav_configuration)" />
-  </xacro:if> -->
-  <!-- <gazebo>
+  </xacro:if>
+  <gazebo>
     <plugin name="gazebo_ros_control" filename="libgazebo_ros_control.so">
       <robotNamespace>$(arg robot_namespace)</robotNamespace>
@@ -357,8 +361,8 @@
       <drift>0.0001 0.0001 0.0001</drift>
     </plugin>
-  </gazebo> -->
+  </gazebo>
   <!-- Optional custom includes. -->
-  <!-- <xacro:include filename="$(arg urdf_extras)" /> -->
+  <xacro:include filename="$(arg urdf_extras)" />
   <!-- Optional for Clearpath internal softwares -->
-  <!-- <xacro:include filename="$(arg cpr_urdf_extras)" /> -->
+  <xacro:include filename="$(arg cpr_urdf_extras)" />
 </robot>

File: robot_description/urdf/custom_description.urdf.xacro (robot description, xacro)
@@ -13,28 +13,3 @@
   <!-- 3) GPS 추가 -->
   <xacro:include filename="$(find robot_description)/urdf/gps.urdf.xacro"/>
-  <!-- 4) Husky Differential Drive Plugin (Gazebo 표준) -->
-  <gazebo>
-    <plugin name="differential_drive_controller" filename="libgazebo_ros_diff_drive.so">
-      <updateRate>50.0</updateRate>
-      <!-- Wheel joints -->
-      <leftJoint>front_left_wheel</leftJoint>
-      <leftJoint>rear_left_wheel</leftJoint>
-      <rightJoint>front_right_wheel</rightJoint>
-      <rightJoint>rear_right_wheel</rightJoint>
-      <!-- Kinematics -->
-      <wheelSeparation>0.5708</wheelSeparation>
-      <wheelDiameter>0.3302</wheelDiameter>
-      <wheelTorque>200</wheelTorque>
-      <!-- Topics -->
-      <commandTopic>husky_velocity_controller/cmd_vel</commandTopic>
-      <odometryTopic>husky_velocity_controller/odom</odometryTopic>
-      <!-- Frames -->
-      <odometryFrame>odom</odometryFrame>
-      <robotBaseFrame>base_link</robotBaseFrame>
-      <!-- Publish odom TF -->
-      <publishOdomTF>$(arg publish_odom_tf)</publishOdomTF>
-      <publishWheelTF>false</publishWheelTF>
-      <publishWheelJointState>false</publishWheelJointState>
-    </plugin>
-  </gazebo>
 </robot>
